File: pcb/lm2596_breakout/lm2596_breakout.kicad_pcb (KiCad board)
At the start: 2 copper layers, 13 parts, among them J1 Conn_01x04, J2 Conn_01x04, J3 Conn_01x04, J4 Conn_01x04, U1 NATIONALSEMI_LM2596SX-ADJ

Commit message: Rough layout + silkscreen.
Parts:
- removed C3: TDK_C3216X5R1E336M160AC, Capacitors_SMD:C_1206
- added G***: LOGO, DBLS_LOGO:van_logo_small, B.Cu at (69.6, 118.1)
- added G***: LOGO, DBLS_LOGO:Rooster_4mmx4mm, F.Cu at (57.4, 127.5)
- C1: value PANASONIC_EEU-EB2E101 -> RUBYCON_100ZLH100MEFC10X20; footprint Capacitors_THT:CP_Radial_D16.0mm_P7.50mm -> Capacitors_THT:CP_Radial_D10.0mm_P5.00mm
- J1, J2, J3, J4: moved to B.Cu
- moved RV1 103.2 mm to (76.7, 119.1), turned to 180 degrees
- moved D1 89.8 mm to (55.4, 118.1), turned to 180 degrees
- moved J4 84.6 mm to (53.3, 132.1)
- moved C2 77.6 mm to (79.0, 104.9), turned to 270 degrees
- moved U1 77.2 mm to (66.0, 125.2), turned to 270 degrees
- moved R2 73.3 mm to (86.4, 118.1), turned to 90 degrees
- moved C1 69.9 mm to (78.5, 126.2), turned to 270 degrees
- moved J2 66.7 mm to (53.3, 111.8)
- moved R1 62.7 mm to (71.4, 106.2), turned to 90 degrees
- moved L1 62.3 mm to (62.0, 108.7), turned to 90 degrees
- moved J1 52.3 mm to (86.4, 132.1)
- moved J3 42.1 mm to (86.4, 111.8)
Connections:
- J1 pad 1: VIN -> GND
- J1 pad 2: VIN -> GND
- J1 pad 3: GND -> VIN
- J1 pad 4: GND -> VIN
- J2 pad 1: /ENABLE -> GND
- J2 pad 3: Net-(J2-Pad3) -> /ISNS_HIGH
- J2 pad 4: GND -> VCC
- J3 pad 1: VCC -> GND
- J3 pad 2: VCC -> GND
- J3 pad 3: GND -> VCC
- J3 pad 4: GND -> VCC
- J4 pad 1: /V_FB -> GND
- J4 pad 2: /ISNS_HIGH -> Net-(J4-Pad2)
- J4 pad 3: VCC -> /ENABLE
- J4 pad 4: GND -> /V_FB
Other:
- board outline added: 38.1 x 33 mm
- board text added: "+"
- board text added: "-"
- board text added: "EN"
- board text added: "FB"
- board text added: "GND"
- board text added: "OUT"
- board text added: "SENSE"
- board text added: "VIN"
- board text added: "VOUT"

Commit message: layout + bom completed.
Parts:
- moved R2 1.52 mm to (86.4, 116.6)
- moved G*** 0.92 mm to (56.9, 128.3)
Connections:
- U1 pad 6: (no net) -> GND
Routing:
- net /V_FB: track 0.00 -> 36.8 mm
- net VCC: track 0.00 -> 32.7 mm, vias 0 -> 1
- net GND: track 0.00 -> 26.2 mm, vias 0 -> 79
- net /ENABLE: track 0.00 -> 17.0 mm
- net /ISNS_HIGH: track 0.00 -> 10.6 mm
- net Net-(D1-Pad1): track 0.00 -> 10.5 mm
- net Net-(R2-Pad1): track 0.00 -> 5.61 mm
- net VIN: vias 0 -> 16
- added copper zone on F.Cu, net /ISNS_HIGH
- added copper zone on B.Cu, net GND
- added copper zone on F.Cu, net GND
- added copper zone on F.Cu, net Net-(D1-Pad1)
- added copper zone on F.Cu, net VCC
- added copper zone on B.Cu, net VIN
- added copper zone on F.Cu, net VIN

Commit message: v1 - placed order with OSH park
Parts:
- removed G***: LOGO, DBLS_LOGO:van_logo_small
- removed G***: LOGO, DBLS_LOGO:Rooster_4mmx4mm
- added C3: MURATA_GCM155R71E103KA37D, Capacitors_SMD:C_0402, B.Cu at (78.7, 118.6)
- added LOGO1: DBLS_Chicken_Small, DBLS_LOGO:Rooster_4mmx4mm, F.Cu at (57.1, 130.3)
- added LOGO2: DBLS_van_logo_small_v1, DBLS_LOGO:van_logo_small, B.Cu at (69.8, 118.1)
- added R1: VISHAYDALE_CRCW04021M00FKEDC, Resistors_SMD:R_0402, F.Cu at (77.2, 117.6)
- added R2: VISHAYDALE_CRCW040268K0FKEDC, Resistors_SMD:R_0402, F.Cu at (77.7, 115.3)
- added R3: VISHAYDALE_CRCW0402150KFKEDC, Resistors_SMD:R_0402, F.Cu at (57.7, 122.4)
- renumbered R1 to R4, R2 to R5
Connections:
- J4 pad 4: /V_FB -> /V_FB_CTRL
Routing:
- net /V_FB_CTRL: track 0.00 -> 4.71 mm
- net VCC: track 32.7 -> 34.4 mm
- net /V_FB: track 36.8 -> 36.3 mm
- net GND: vias 79 -> 82
