File: pcb/lm2596_breakout/lm2596_breakout.sch (KiCad schematic (older format))
At the start: 13 parts, among them J1 Conn_01x04, J2 Conn_01x04, J3 Conn_01x04, J4 Conn_01x04, U1 NATIONALSEMI_LM2596SX-ADJ

Commit message: Rough layout + silkscreen.
Parts:
- removed C1: PANASONIC_EEU-EB2E101, Capacitors_THT:CP_Radial_D16.0mm_P7.50mm, symbol DBLS_Capacitor:PANASONIC_EEU-EB2E101
- removed C3: TDK_C3216X5R1E336M160AC, Capacitors_SMD:C_1206, symbol DBLS_Capacitor:TDK_C3216X5R1E336M160AC
- added C1: RUBYCON_100ZLH100MEFC10X20, Capacitors_THT:CP_Radial_D10.0mm_P5.00mm, symbol DBLS_Capacitor:RUBYCON_100ZLH100MEFC10X20
Connections:
- net ENABLE: now also J4.3 (Pin_3); no longer J2.1 (Pin_1)
- net GND: now also J1.1 (Pin_1), J1.2 (Pin_2), J2.1 (Pin_1), J3.1 (Pin_1), J3.2 (Pin_2), J4.1 (Pin_1), C1.2; no longer J1.3 (Pin_3), J1.4 (Pin_4), J2.4 (Pin_4), J3.3 (Pin_3), J3.4 (Pin_4), J4.4 (Pin_4)
- net ISNS_HIGH: now also J2.3 (Pin_3); no longer J4.2 (Pin_2)
- net VCC: now also J2.4 (Pin_4), J3.3 (Pin_3), J3.4 (Pin_4); no longer J3.1 (Pin_1), J3.2 (Pin_2), J4.3 (Pin_3)
- net VIN: now also J1.3 (Pin_3), J1.4 (Pin_4), C1.1; no longer J1.1 (Pin_1), J1.2 (Pin_2)
- net V_FB: now also J4.4 (Pin_4); no longer J4.1 (Pin_1)
Changed lines of the file:
@@
 	6900 1950 6900 1850
 Connection ~ 6900 1850
-Wire Wire Line
-	6900 1850 7300 1850
-Wire Wire Line
-	7300 1950 7300 1850
-Connection ~ 7300 1850
 $Comp
 L power:GND #PWR0105
@@
 F 3 "" H 6900 2100 50  0001 C CNN
 	1    6900 2100
-	1    0    0    -1
-$EndComp
-$Comp
-L power:GND #PWR0106
-U 1 1 61F68CE4
-P 7300 2100
-F 0 "#PWR0106" H 7300 1850 50  0001 C CNN
-F 1 "GND" H 7300 1950 50  0000 C CNN
-F 2 "" H 7300 2100 50  0001 C CNN
-F 3 "" H 7300 2100 50  0001 C CNN
-	1    7300 2100
 	1    0    0    -1
 $EndComp
@@
 L SparkFun-Aesthetics:VCC #SUPPLY0102
 U 1 1 61FA9655
-P 7900 1750
-F 0 "#SUPPLY0102" H 7900 1750 50  0001 L BNN
-F 1 "VCC" H 7860 1890 50  0000 L BNN
-F 2 "" H 7900 1750 50  0001 C CNN
-F 3 "" H 7900 1750 50  0001 C CNN
-	1    7900 1750
-	1    0    0    -1
-$EndComp
-Wire Wire Line
-	7900 1750 7900 1850
+P 7000 1750
+F 0 "#SUPPLY0102" H 7000 1750 50  0001 L BNN
+F 1 "VCC" H 6960 1890 50  0000 L BNN
+F 2 "" H 7000 1750 50  0001 C CNN
+F 3 "" H 7000 1750 50  0001 C CNN
+	1    7000 1750
+	1    0    0    -1
+$EndComp
+Wire Wire Line
+	7000 1750 7000 1850
 Wire Wire Line
 	5550 1850 5750 1850
@@
 Wire Wire Line
 	4750 4150 4750 4050
-Wire Wire Line
-	4900 5150 4200 5150
-Text Label 4200 5150 0    50   ~ 0
+Text Label 6000 5250 0    50   ~ 0
 ENABLE
 $Comp
@@
 L Connector_Generic:Conn_01x04 J1
 U 1 1 61FD15A2
-P 5100 4250
-F 0 "J1" H 5100 4450 50  0000 C CNN
-F 1 "Conn_01x04" H 5100 3950 50  0000 C CNN
-F 2 "Pin_Headers:Pin_Header_Straight_1x04_Pitch2.54mm" H 5100 4250 50  0001 C CNN
-F 3 "~" H 5100 4250 50  0001 C CNN
-	1    5100 4250
-	1    0    0    -1
+P 5100 4350
+F 0 "J1" H 5100 4550 50  0000 C CNN
+F 1 "Conn_01x04" H 5100 4050 50  0000 C CNN
+F 2 "Pin_Headers:Pin_Header_Straight_1x04_Pitch2.54mm" H 5100 4350 50  0001 C CNN
+F 3 "~" H 5100 4350 50  0001 C CNN
+	1    5100 4350
+	1    0    0    1
 $EndComp
 Wire Wire Line
@@
 Text Label 6000 1400 0    50   ~ 0
 ISNS_HIGH
-Text Label 6000 5350 0    50   ~ 0
+Text Label 4400 5150 0    50   ~ 0
 ISNS_LOW
-Text Label 6000 5250 0    50   ~ 0
+Text Label 4400 5250 0    50   ~ 0
 ISNS_HIGH
 $Comp
@@
 	6000 5450 6000 5500
 Wire Wire Line
-	6000 5350 5850 5350
-Wire Wire Line
-	5850 5250 6000 5250
-Wire Wire Line
 	6000 5150 5850 5150
-NoConn ~ 4900 5250
-NoConn ~ 4900 5350
+NoConn ~ 5850 5350
 $Comp
 L DBLS_Diode:VISHAY_SSA34HE3_A_I D1
@@
 $EndComp
 $Comp
-L DBLS_Capacitor:TDK_C3216X5R1E336M160AC C3
-U 1 1 61FB0D92
-P 7300 2050
-F 0 "C3" H 7350 2125 40  0000 L CNN
-F 1 "TDK_C3216X5R1E336M160AC" H 6850 2900 50  0001 L CNN
-F 2 "Capacitors_SMD:C_1206" H 7300 2400 50  0001 C CNN
-F 3 "" H 7300 2275 20  0001 C CNN
-F 4 "33uF" H 7400 2000 30  0000 C CNN "capacitance"
-F 5 "TDK Corporation" H 7300 2800 50  0001 C CNN "mfg"
-F 6 "C3216X5R1E336M160AC" H 7300 2700 50  0001 C CNN "mfg_pn"
-F 7 "Digikey" H 7300 2600 50  0001 C CNN "vendor"
-F 8 "445-8046-2-ND" H 7300 2500 50  0001 C CNN "vendor_pn"
-F 9 "YES" H 7225 2125 20  0001 C CNN "place"
-F 10 "CAP CER 33UF 25V X5R 1206" H 7300 2050 50  0001 C CNN "description"
-	1    7300 2050
-	1    0    0    -1
-$EndComp
-$Comp
 L Connector_Generic:Conn_01x04 J2
 U 1 1 61FB781F
-P 5100 5250
-F 0 "J2" H 5100 5450 50  0000 C CNN
-F 1 "Conn_01x04" H 5100 4950 50  0000 C CNN
-F 2 "Pin_Headers:Pin_Header_Straight_1x04_Pitch2.54mm" H 5100 5250 50  0001 C CNN
-F 3 "~" H 5100 5250 50  0001 C CNN
-	1    5100 5250
-	1    0    0    -1
+P 5100 5350
+F 0 "J2" H 5100 5550 50  0000 C CNN
+F 1 "Conn_01x04" H 5100 5050 50  0000 C CNN
+F 2 "Pin_Headers:Pin_Header_Straight_1x04_Pitch2.54mm" H 5100 5350 50  0001 C CNN
+F 3 "~" H 5100 5350 50  0001 C CNN
+	1    5100 5350
+	1    0    0    1
 $EndComp
 $Comp
 L Connector_Generic:Conn_01x04 J4
 U 1 1 61FB8504
-P 5650 5250
-F 0 "J4" H 5650 5450 50  0000 C CNN
-F 1 "Conn_01x04" H 5650 4950 50  0000 C CNN
-F 2 "Pin_Headers:Pin_Header_Straight_1x04_Pitch2.54mm" H 5650 5250 50  0001 C CNN
-F 3 "~" H 5650 5250 50  0001 C CNN
-	1    5650 5250
-	-1   0    0    -1
+P 5650 5350
+F 0 "J4" H 5650 5550 50  0000 C CNN
+F 1 "Conn_01x04" H 5650 5050 50  0000 C CNN
+F 2 "Pin_Headers:Pin_Header_Straight_1x04_Pitch2.54mm" H 5650 5350 50  0001 C CNN
+F 3 "~" H 5650 5350 50  0001 C CNN
+	1    5650 5350
+	-1   0    0    1
 $EndComp
 $Comp
 L Connector_Generic:Conn_01x04 J3
 U 1 1 61FB8C13
-P 5650 4250
-F 0 "J3" H 5650 4450 50  0000 C CNN
-F 1 "Conn_01x04" H 5650 3950 50  0000 C CNN
-F 2 "Pin_Headers:Pin_Header_Straight_1x04_Pitch2.54mm" H 5650 4250 50  0001 C CNN
-F 3 "~" H 5650 4250 50  0001 C CNN
-	1    5650 4250
-	-1   0    0    -1
+P 5650 4350
+F 0 "J3" H 5650 4550 50  0000 C CNN
+F 1 "Conn_01x04" H 5650 4050 50  0000 C CNN
+F 2 "Pin_Headers:Pin_Header_Straight_1x04_Pitch2.54mm" H 5650 4350 50  0001 C CNN
+F 3 "~" H 5650 4350 50  0001 C CNN
+	1    5650 4350
+	-1   0    0    1
 $EndComp
 $Comp
@@
 Wire Wire Line
 	3200 3000 3350 3000
-Wire Wire Line
-	7300 1850 7900 1850
 $Comp
 L SparkFun-Aesthetics:VCC #SUPPLY0106
@@
 Vout: 1.23V to 21V
 $Comp
-L DBLS_Capacitor:PANASONIC_EEU-EB2E101 C1
-U 1 1 61FDD64F
+L DBLS_Capacitor:RUBYCON_100ZLH100MEFC10X20 C1
+U 1 1 61FAB912
 P 3250 1800
 F 0 "C1" H 3300 1875 40  0000 L CNN
-F 1 "PANASONIC_EEU-EB2E101" H 2800 2650 50  0001 L CNN
-F 2 "Capacitors_THT:CP_Radial_D16.0mm_P7.50mm" H 3250 2150 50  0001 C CNN
+F 1 "RUBYCON_100ZLH100MEFC10X20" H 2800 2650 50  0001 L CNN
+F 2 "Capacitors_THT:CP_Radial_D10.0mm_P5.00mm" H 3250 2150 50  0001 C CNN
 F 3 "" H 3250 2025 20  0001 C CNN
 F 4 "100uF" H 3350 1750 30  0000 C CNN "capacitance"
-F 5 "Panasonic Electronic Components" H 3250 2550 50  0001 C CNN "mfg"
-F 6 "EEU-EB2E101" H 3250 2450 50  0001 C CNN "mfg_pn"
+F 5 "Rubycon" H 3250 2550 50  0001 C CNN "mfg"
+F 6 "100ZLH100MEFC10X20" H 3250 2450 50  0001 C CNN "mfg_pn"
 F 7 "Digikey" H 3250 2350 50  0001 C CNN "vendor"
-F 8 "P5928-ND" H 3250 2250 50  0001 C CNN "vendor_pn"
+F 8 "1189-1887-ND" H 3250 2250 50  0001 C CNN "vendor_pn"
 F 9 "YES" H 3175 1875 20  0001 C CNN "place"
-F 10 "CAP ALUM 100UF 20% 250V RADIAL" H 3250 1800 50  0001 C CNN "description"
+F 10 "CAP ALUM 100UF 20% 100V RADIAL" H 3250 1800 50  0001 C CNN "description"
 	1    3250 1800
 	1    0    0    -1
 $EndComp
+Wire Wire Line
+	5850 5250 6000 5250
+NoConn ~ 4900 5350
+Wire Wire Line
+	6900 1850 7000 1850
+Wire Wire Line
+	4400 5150 4900 5150
+Wire Wire Line
+	4900 5250 4400 5250
 $EndSCHEMATC

Commit message: layout + bom completed.
Connections:
- net GND: now also U1.6 (GND)
Changed lines of the file:
@@
 Wire Wire Line
 	4900 5250 4400 5250
+$Comp
+L power:GND #PWR?
+U 1 1 6201796D
+P 4650 2050
+F 0 "#PWR?" H 4650 1800 50  0001 C CNN
+F 1 "GND" H 4650 1900 50  0001 C CNN
+F 2 "" H 4650 2050 50  0001 C CNN
+F 3 "" H 4650 2050 50  0001 C CNN
+	1    4650 2050
+	1    0    0    -1
+$EndComp
 $EndSCHEMATC

Commit message: v1 - placed order with OSH park
Parts:
- added C3: MURATA_GCM155R71E103KA37D, Capacitors_SMD:C_0402, symbol DBLS_Capacitor:MURATA_GCM155R71E103KA37D
- added LOGO1: DBLS_Chicken_Small, DBLS_LOGO:Rooster_4mmx4mm, symbol DBLS_Logo:DBLS_Chicken_Small
- added LOGO2: DBLS_van_logo_small_v1, DBLS_LOGO:van_logo_small, symbol DBLS_Logo:DBLS_van_logo_small_v1
- added R1: VISHAYDALE_CRCW04021M00FKEDC, Resistors_SMD:R_0402, symbol DBLS_Resistor:VISHAYDALE_CRCW04021M00FKEDC
- added R2: VISHAYDALE_CRCW040268K0FKEDC, Resistors_SMD:R_0402, symbol DBLS_Resistor:VISHAYDALE_CRCW040268K0FKEDC
- added R3: VISHAYDALE_CRCW0402150KFKEDC, Resistors_SMD:R_0402, symbol DBLS_Resistor:VISHAYDALE_CRCW0402150KFKEDC
- renumbered R1 to R4, R2 to R5
Connections:
- net GND: now also R2.2
- net VCC: now also C3.1, R1.1
- net V_FB: now also C3.2, R1.2, R2.1, R3.1; no longer J4.4 (Pin_4)
- new net V_FB_CTRL: J4.4 (Pin_4), R3.2
Other:
- note added: "CW to Increase Voltage\nVout: 1.23V to 21V"
- note added: "DAC ADJUSTMENT:"
- note added: "FIXED VOLTAGE:"
- note added: "POT ADJUSTMENT:"
- note added: "VOUT = 1.23V * (1 + R2 / R1)\nR1 = 1M\nR2(3.3V)= 310k\nR2(5V) = 185k\nR2(12V) = 69.8k"
- note added: "VOUT = VREF+ ((VREF / R2) + (VREF - VDAC)/R3) * R1\nR1: 1M\nR2: 68k\nR3: 150k\nVMIN: 0.82V\nVMAX: 17.4V\nVNOM: 12.5V"
- note removed: "CW to Increase Voltage"
- note removed: "VOUT = 1.23V * (1 + R2 / R1)\nR1 = 1k\nR2(3.3V) = 1683\nR2(5V) = 3065\nR2(12V) = 8756"
- note removed: "Vout: 1.23V to 21V"
- moved on the sheet: R5, RV1

Commit message: Updated schematic to include lm2596 on board.
Other:
- note added: "TODO: Consider making these breadboard compatible"
- note added: "TODO: Move R3 to be in parallel with current feedback fet"
- note added: "TODO: Move R4 this to other side of caps"
- note added: "TODO: Update to correct values"
Changed lines of the file:
@@
 	1    0    0    -1
 $EndComp
+Text Notes 5700 1250 0    50   ~ 0
+TODO: Move R4 this to other side of caps
+Text Notes 4950 3200 0    50   ~ 0
+TODO: Move R3 to be in parallel with current feedback fet
+Text Notes 4950 5900 0    50   ~ 0
+TODO: Consider making these breadboard compatible
+Text Notes 8550 1150 0    50   ~ 0
+TODO: Update to correct values
 $EndSCHEMATC
