File: pcb/simpleBuck/power_stage.sch (KiCad schematic (older format))
At the start: 48 parts, among them Q1 TRANSISTOR_PNPMMBT4403, U2 TI_INA181A2, U3 TI_TL072HIDBVR, U4 TI_TL072HIDBVR, U7 NATIONALSEMI_LM2596SX-ADJ

Commit message: Added jumpers and finalized DAC/ADC selection.
Parts:
- removed JP1: PAD_JUMPER_2PIN_NC, DBLS_Misc:PAD_JUMPER_2PIN_NC, symbol DBLS_Misc:PAD_JUMPER_2PIN_NC
- removed JP2, JP3, JP4, JP5, JP6: PAD_JUMPER_2PIN_0603, DBLS_Misc:PAD_JUMPER_2PIN_0603, symbol DBLS_Misc:PAD_JUMPER_2PIN_0603
- removed R15: VISHAYDALE_CRCW0402150KFKEDC, Resistors_SMD:R_0402, symbol DBLS_Resistor:VISHAYDALE_CRCW0402150KFKEDC
- removed RV1, RV2: BOURNS_PV37W203C01B00, Potentiometers:Potentiometer_Trimmer_Bourns_3299Y, symbol DBLS_Resistor:BOURNS_PV37W203C01B00
- removed TP1: DBLS_TESTPOINT_NORMAL, DBLS_Misc:DBLS_Testpoint_Normal, symbol DBLS_Misc:DBLS_TESTPOINT_NORMAL
- added JP3, JP4, JP5, JP7, JP8: PAD_JUMPER_2PIN_NC_BY_TRACE, DBLS_Jumpers:PAD_JUMPER_2PIN_NC_BY_TRACE, symbol DBLS_Misc:PAD_JUMPER_2PIN_NC_BY_TRACE
- added JP6: PAD_JUMPER_2PIN_NO, DBLS_Jumpers:PAD_JUMPER_2PIN_NO_0603, symbol DBLS_Misc:PAD_JUMPER_2PIN_NO
- added R15: VISHAYDALE_CRCW0603150KFKEAC, Resistors_SMD:R_0603, symbol DBLS_Resistor:VISHAYDALE_CRCW0603150KFKEAC
- added R17, R2: VISHAY_CRCW060310K0FKEBC, Resistors_SMD:R_0603, symbol DBLS_Resistor:VISHAY_CRCW060310K0FKEBC
- added TP5, TP6, TP7, TP8, TP9: DBLS_TESTPOINT_NORMAL, DBLS_Misc:DBLS_Testpoint_Normal, symbol DBLS_Misc:DBLS_TESTPOINT_NORMAL
Connections:
- net GND: now also JP3.2, R17.2, R2.2
- net I_ADC: now also U2.1, JP4.1, TP5.1; no longer R6.1
- net VOUT_HI: now also R17.1, R2.1
- net V_ADC: now also R7.1, U3.1, JP5.1, TP6.1; no longer R10.1
- net V_FB: now also JP7.2, JP8.2, TP9.1
- net at C6.1, C8.1, D1.2 (A)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: now also TP7.1
- net at D4.1 (K): now also JP7.1
- net at U2.5 (REF): now also JP3.1
- net at C10.2, D3.1 (K), R10.2: now also U3.5 (+), JP6.1; no longer U3.3 (+)
- net at C10.1, C11.1, D3.2 (A): now also U3.7, R15.1, TP8.1; no longer U3.1
- net at C11.2: now also JP6.2
- net at R11.2: now also U3.6 (-); no longer U3.2 (-)
- net at R3.1, R4.1: now also U3.3 (+); no longer U3.5 (+)
- net at R5.1, R7.2: now also U3.2 (-); no longer U3.6 (-)
- new net: JP4.2, R6.1
- new net: JP5.2, R10.1
- new net: JP8.1, R15.2
Other:
- moved on the sheet: C7
